File: demo/Demo_project/Demo_project.kicad_sch (KiCad schematic)
At the start: 28 parts, among them J1 USB_C_Receptacle_USB2.0, J2 Conn_01x04, J3 Screw_Terminal_01x03, J4 Screw_Terminal_01x08, J5 Screw_Terminal_01x02, K1 RT314A05, Q1 UMH3N, Q2 BC817, SW1 SW_SPST, U1 ESP32-WROOM-32D, U2 USBLC6-2P6, U3 CP2104, U4 Si7021-A20, U5 74HC245, U6 LM1117MP-3.3

Commit message: v0.1
Parts:
- added C2, C5, C8, C9: 22u, symbol Device:C
- added C3, C6: 100n, symbol Device:C
- added C4, C7: 47u, symbol Device:C
- added F2: Polyfuse 1A, symbol Device:Fuse
- added FB1: BLM21PG221, symbol Device:FerriteBead
- added R4: 10k, symbol Device:R
- added R5, R6: 22R, symbol Device:R
- R1: value R -> 660
- U6: value LM1117MP-3.3 -> TLV1117LV-3.3
Connections:
- net +3.3V: now also C9.1
- net +5V: now also U2.5 (VBUS), U3.7 (REGIN), U3.8 (VBUS), C2.1, C3.1, C4.1, C8.1, F2.2
- net GND: now also U2.2 (GND), U3.2 (GND), U3.25 (GND), U6.1 (GND), C2.2, C3.2, C4.2, C5.2, C6.2, C7.2, C8.2, C9.2
- net RTS: now reaches Q1.3 (C2)
- net RTS: now also Q1.2 (B1), U3.19 (~{RTS})
- net EN: now reaches Q1.4 (E2)
- net DTR: now reaches Q1.5 (B2)
- net DTR: now also Q1.1 (E1), U3.23 (~{DTR})
- net at J1.A6 (D+), J1.B6 (D+): now also U2.3 (I/O2); no longer U2.1 (I/O1)
- net at U2.4 (I/O2): now also U3.3 (D+)
- net at J1.A7 (D-), J1.B7 (D-): now also U2.1 (I/O1); no longer U2.6 (I/O1)
- net at U3.16 (VPP): now also C7.1
- net at U3.20 (RXD): now also R6.1
- net at U3.21 (TXD): now also R5.1
- net at U3.4 (D-): now also U2.6 (I/O1)
- net +3.3VA: now reaches U3.5 (VIO)
- net +3.3VA: now also U3.6 (VDD), C5.1, C6.1, R4.1
- net at U3.9 (~{RST}): now also R4.2
- net IO0: now reaches Q1.6 (C1)
- net IO0: now also U1.25 (IO0)
- net +5VP: now reaches J1.A4 (VBUS), J1.A9 (VBUS), J1.B4 (VBUS), J1.B9 (VBUS)
- net +5VP: now also FB1.1
- net RX: now reaches U1.34 (RXD0/IO3)
- net RX: now also R5.2
- net TX: now reaches U1.35 (TXD0/IO1)
- net TX: now also R6.2
- new net: F2.1, FB1.2
Other:
- moved on the sheet: D4, J1, Q1A, Q1B, R1, R2, R3, U2, U3

Commit message: Beta
Parts:
- added C10, C12, C13: 100n, symbol Device:C
- added C11: 22u, symbol Device:C
- added R10, R8, R9: 1k, symbol Device:R
- added R11, R12: 4K7, symbol Device:R
- added R13, R14: 10K, symbol Device:R
- added R15: 1K, symbol Device:R
- added R16, R17, R18, R19: 22, symbol Device:R
- added R7: 10k, symbol Device:R
- C1: value C_Polarized -> 1000u/25V
- D3: value LED -> YELLOW
- U5: value 74HC245 -> 74AHCT245
Connections:
- net +3.3V: now also D1.4 (A), J2.2 (Pin_2), U4.5 (VDD), C11.1, C12.1, R11.1, R12.1, R7.1
- net +5V: now also D2.1 (K), K1.A1, U5.1 (A->B), U5.20 (VCC), C13.1, R15.1
- net GND: now also C1.2, H1.1, H2.1, H3.1, H4.1, J2.1 (Pin_1), J5.2 (Pin_2), Q2.2 (E), SW1.1 (A), U4.2 (GND), U4.7 (PAD), U5.10 (GND), U5.19 (CE), U5.6 (A4), U5.7 (A5), U5.8 (A6), U5.9 (A7), C10.2, C11.2, C12.2, C13.2, R13.2
- net at J5.1 (Pin_1): now also C1.1, F1.1
- net at Q2.1 (B): now also R13.1, R14.2
- net at Q2.3 (C): now also D2.2 (A), D3.1 (K), K1.A2
- net SDA: now reaches J2.3 (Pin_3)
- net SDA: now also U4.1 (SDA), R11.2
- net SCL: now reaches J2.4 (Pin_4)
- net SCL: now also U4.6 (SCL), R12.2
- net at J3.1 (Pin_1): now also K1.12
- net at J3.2 (Pin_2): now also K1.11
- net at J3.3 (Pin_3): now also K1.14
- net at J4.1 (Pin_1): now also F1.2, J4.2 (Pin_2)
- net at J4.3 (Pin_3): now also R16.2
- net at J4.4 (Pin_4): now also R17.2
- net at J4.5 (Pin_5): now also R18.2
- net at J4.6 (Pin_6): now also R19.2
- net at D1.1 (RK): now also R8.1
- net at D1.2 (GK): now also R9.2
- net at D1.3 (BK): now also R10.2
- net SW: now reaches SW1.2 (B)
- net SW: now also C10.1, R7.2
- net at U5.15 (B3): now also R19.1
- net at U5.16 (B2): now also R18.1
- net at U5.17 (B1): now also R17.1
- net at U5.18 (B0): now also R16.1
- net LEDSTR1: now reaches U5.2 (A0)
- net LEDSTR2: now reaches U5.3 (A1)
- net LEDSTR3: now reaches U5.4 (A2)
- net LEDSTR4: now reaches U5.5 (A3)
- net at D3.2 (A): now also R15.2
- new net LED_B: R10.1
- new net LED_G: R9.1
- new net LED_R: R8.2
- new net RELAY: R14.1
- no-connect marks 0 -> 4
Other:
- note added: "GND"
- note added: "SCL"
- note added: "SDA"
- note added: "VCC"
- moved on the sheet: C1, D1, D2, D3, F1, J2, J3, J4, J5, K1, Q2, SW1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

Commit message: v0.1 beta
Parts:
- added C14, C16: 100n, symbol Device:C
- added C15: 22u, symbol Device:C
- added R20: 10K, symbol Device:R
Connections:
- net +3.3V: now also U1.2 (VDD), C14.1, C15.1, R20.1
- net EN: now also U1.3 (EN), C16.1, R20.2
- net GND: now also U1.1 (GND), U1.15 (GND), U1.38 (GND), U1.39 (GND), C14.2, C15.2, C16.2
- net LEDSTR1: now also U1.27 (IO16)
- net LEDSTR2: now also U1.28 (IO17)
- net LEDSTR3: now also U1.30 (IO18)
- net LEDSTR4: now also U1.31 (IO19)
- net LED_B: now also U1.23 (IO15)
- net LED_G: now also U1.13 (IO14)
- net LED_R: now also U1.16 (IO13)
- net RELAY: now also U1.33 (IO21)
- net SCL: now also U1.37 (IO23)
- net SDA: now also U1.36 (IO22)
- no-connect marks 4 -> 20
Other:
- moved on the sheet: U1
